File: PCB/NaviCore_V1/NaviCore_V1.kicad_pcb (KiCad board)
At the start: 2 copper layers, 65.2 x 84.8 mm, 9 parts, among them J1 SBUS_IN, J2 SBUS_OUT, J3 MAESTRO, J4 SERIAL_1, J5 SEREIAL_2, J6 SERIAL_3, J7 Screw_Terminal_01x02, U1 ESP32-S3-DEVKITC-1-N8R2

Commit message: updates
Parts:
- added G***: LOGO, 01-Custom:NC_Name8High, F.Cu at (152.6, 120.4)
- added G***: LOGO, 01-Custom:NaviCoreLogo_Solo_15, F.Cu at (172.7, 117.4)
- added G***: LOGO, 01-Custom:R2_Logo_V2, F.Cu at (122.5, 119.6)
- added G***: LOGO, 01-Custom:NC_Name8High, B.Cu at (183.3, 101.3)
- added G***: LOGO, 01-Custom:qr_code_20, B.Cu at (147.7, 89.5)
- added H1: MountingHole, MountingHole:MountingHole_3.2mm_M3, F.Cu at (185.0, 56.5)
- added H2: MountingHole, MountingHole:MountingHole_3.2mm_M3, F.Cu at (137.0, 56.5)
- added H3: MountingHole, MountingHole:MountingHole_3.2mm_M3, F.Cu at (185.0, 121.2)
- added H4: MountingHole, MountingHole:MountingHole_3.2mm_M3, F.Cu at (137.0, 121.1)
- moved J7 54.4 mm to (176.6, 63.7), turned to 180 degrees
- moved J1 27.0 mm to (176.1, 73.2), turned to -90 degrees
- moved J2 21.9 mm to (176.1, 79.3), turned to -90 degrees
- moved J6 17.2 mm to (176.1, 108.5)
- moved J5 13.9 mm to (176.1, 100.4)
- moved R1 11.9 mm to (166.1, 69.7)
- moved J4 10.6 mm to (176.1, 92.3)
- moved J3 8.65 mm to (176.1, 85.5)
Connections:
- U1 pad J3_10: unconnected-(U1-GPIO38-PadJ3_10) -> SERIAL_3_TX
- U1 pad J3_16: SERIAL_3_TX -> unconnected-(U1-GPIO48-PadJ3_16)
Routing:
- net MAESTRO_RX: track 0.00 -> 40.0 mm
- net MAESTRO_TX: track 0.00 -> 39.1 mm
- net SBUS_OUT: track 0.00 -> 37.8 mm
- net SERIAL_1_RX: track 0.00 -> 37.1 mm
- net SBUS_IN: track 0.00 -> 36.3 mm
- net 3.3V: track 0.00 -> 34.8 mm
- net SERIAL_2_TX: track 0.00 -> 33.7 mm
- net SERIAL_1_TX: track 0.00 -> 33.7 mm
- net SERIAL_3_TX: track 0.00 -> 30.5 mm
- net Net-(U1-GPIO0): track 0.00 -> 22.8 mm
- net SERIAL_3_RX: track 0.00 -> 22.3 mm
- net SERIAL_2_RX: track 0.00 -> 14.1 mm
- net GND: track 0.00 -> 7.62 mm
- net unconnected-(U1-U0TXD/GPIO43-PadJ3_2): track 0.00 -> 2.55 mm
- net unconnected-(U1-USB_D-/GPIO19-PadJ3_20): track 0.00 -> 2.54 mm
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- added copper zone on F.Cu, net 5V
- added copper zone on B.Cu, net GND
Other:
- board size 65.2 x 84.8 mm -> 55.1 x 71.7 mm
- board text added: "5V"
- board text added: "5v"
- board text added: "G"
- board text added: "MAESTRO"
- board text added: "Rx"
- board text added: "S"
- board text added: "SBUS IN"
- board text added: "SBUS OUT"
- board text added: "SERIAL 1"
- board text added: "SERIAL 2"
- board text added: "SERIAL 3"
- board text added: "Tx"
- board text added: "v1.0"
- board text added: "ver: 1.0 date: 18 jun 26 created by: greg hulette"
